File: PCB/RGBSegment/RGBSegment/RGBSegment.kicad_sch (KiCad schematic)
At the start: 93 parts

Commit message: linear display test.
Parts:
- removed TP?: PB7_TP, TestPoint:TestPoint_Pad_1.0x1.0mm, symbol Connector:TestPoint
- added C? (x3): 10uF, Capacitor_SMD:C_0402_1005Metric, symbol Device:C_Small
- added C? (x4): 22uF, symbol Device:C_Small
- added C?: 100nF, Capacitor_SMD:C_0402_1005Metric, symbol Device:C_Small
- added C?: 1uF, symbol Device:C_Small
- added D?: Heartbeat, symbol Device:LED_Small
- added J?: Right, symbol Connector_Generic:Conn_01x04
- added J?: Top, symbol Connector_Generic:Conn_01x04
- added J?: Left, symbol Connector_Generic:Conn_01x04
- added J?: Bottom, symbol Connector_Generic:Conn_01x04
- added JP?: Jumper_2_Open, symbol Jumper:Jumper_2_Open
- added L?: 1uH, symbol Device:L_Small
- added R?: 120, symbol Device:R_Small
- added R?: 330, symbol Device:R_Small
- added R?: 10k, symbol Device:R_Small
- added R?: 1M, Resistor_SMD:R_0402_1005Metric, symbol Device:R_Small
- added U?: HT75xx-1-SOT89, Package_TO_SOT_SMD:SOT-89-3, symbol Regulator_Linear:HT75xx-1-SOT89
- added U?: MIC2877-AYFT-TR, SnapEDA Library:VREG_MIC2877-AYFT-TR, symbol MIC2877-AYFT-TR:MIC2877-AYFT-TR
- added U?: SN65HVD230DRG4, SnapEDA Library:SOIC127P599X175-8N, symbol SN65HVD230DRG4:SN65HVD230DRG4
- U? (x49): MANUFACTURER Worldsemi -> (none); STANDARD Manufacturer Recommendations -> (none)
Connections:
- net +3V3: now also C?.1, C?.1, C?.1, U?.3 (VCC), U?.3 (VOUT)
- net +5V: now also C?.1, C?.1, C?.1, C?.1, U?.2 (VIN), U?.5 (VOUT), U?.7 (FB)
- net GND: now also C?.2, C?.2, C?.2, C?.2, C?.2, C?.2, C?.2, C?.2, C?.2, J?.4 (Pin_4), J?.4 (Pin_4), J?.4 (Pin_4), J?.4 (Pin_4), R?.2, U?.1 (GND), U?.2 (AGND), U?.2 (GND), U?.3 (PGND)
- net at U?.28 (PF0): now also D?.2 (A)
- net USB0DM: no longer names the net of U?.43 (PD4)
- net USB0DP: no longer names the net of U?.44 (PD5)
- net USB0ID: no longer names the net of U?.45 (PB0/USB0ID)
- net USB0VBUS: no longer names the net of U?.46 (PB1/USB0VBUS)
- new net: JP?.1 (A), R?.1
- new net: L?.2, U?.4 (SW)
- new net: R?.2, U?.6 (EN)
- new net: R?.2, U?.8 (PG)
- new net: D?.1 (K), R?.1
- new net +5VA: C?.1, C?.1, J?.3 (Pin_3), J?.3 (Pin_3), J?.3 (Pin_3), J?.3 (Pin_3), L?.1, R?.1, R?.1, U?.1 (VIN)
- new net CANH: J?.1 (Pin_1), J?.1 (Pin_1), J?.1 (Pin_1), J?.1 (Pin_1), JP?.2 (B), U?.7 (CANH)
- new net CANL: J?.2 (Pin_2), J?.2 (Pin_2), J?.2 (Pin_2), J?.2 (Pin_2), R?.2, U?.6 (CANL)
- new net CAN_MODE: U?.8 (RS)
- new net CAN_RX: U?.4 (R)
- new net CAN_TX: U?.1 (D)
- no-connect marks 27 -> 2
Other:
- note added: "5V-3V3 Regulator"
- note added: "5V-5V Regulator"
- note added: "CAN Transceiver"
- note added: "Connectors and Mounting Holes"
- note added: "LEDs"
- note added: "Photoresistors"
- note added: "TODO: - components table - opt ESP8266 port - review schematic - layout"
- note added: "Testpoints"
- note removed: "External LED sanity debug."
- note removed: "TODO: 12V - 5V Switching Regulator 5V - 3.3 Linear Regulator Signals for photoresistors, CAN bus for controllers, connector for SDO another RGBSegment and controller override header"
- moved on the sheet: C?, J?, R?, SW?, TP?, U?, Y?
